Commit message: Commit before leaving

File: source/extensions/omni.isaac.lab_tasks/omni/isaac/lab_tasks/direct/stewart/urdf/Stewart.urdf (robot description, URDF)
Before this commit: robot modified_stewart, 13 links, 12 joints
Links:
- link foot0: geometry collision cylinder length=0.0550 radius=0.03; visual cylinder length=0.0550 radius=0.03
- link foot1: geometry collision cylinder length=0.0550 radius=0.03; visual cylinder length=0.0550 radius=0.03
- link foot2: geometry collision cylinder length=0.0550 radius=0.03; visual cylinder length=0.0550 radius=0.03
- link intermediate_link0: geometry visual box size=0.01 0.01 0.004
- link intermediate_link1: geometry visual box size=0.001 0.001 0.004
- link intermediate_link2: geometry visual box size=0.001 0.001 0.004
- link lower_leg0: geometry visual cylinder length=0.0496 radius=0.01
- link lower_leg1: geometry visual cylinder length=0.0496 radius=0.01
- link lower_leg2: geometry visual cylinder length=0.0496 radius=0.01
- link plane: geometry collision box size=0.18 0.18 0.0215; visual box size=0.18 0.18 0.0215
- link upper_leg0: geometry visual cylinder length=0.0623 radius=0.01
- link upper_leg1: geometry visual cylinder length=0.0623 radius=0.01
- link upper_leg2: geometry visual cylinder length=0.0623 radius=0.01
Joints:
- joint foot_joint0: limit lower=0 upper=1.1 effort=300 velocity=0.1 -> lower=0 upper=1.6 effort=300 velocity=0.1; origin xyz=0 0 -0.1 -> xyz=0 0 -0.0496
- joint foot_joint1: limit lower=0 upper=1.1 effort=300 velocity=0.1 -> lower=0 upper=1.6 effort=300 velocity=0.1; origin xyz=0 0 -0.1 -> xyz=0 0 -0.0496
- joint foot_joint2: limit lower=0 upper=1.1 effort=300 velocity=0.1 -> lower=0 upper=1.6 effort=300 velocity=0.1; origin xyz=0 0 -0.1 -> xyz=0 0 -0.0496
- joint lower_leg_joint0: limit lower=0 upper=2.1 effort=300 velocity=0.1 -> lower=0 upper=3.1 effort=300 velocity=0.1; origin xyz=0 0 -0.1 -> xyz=0 0 -0.0623
- joint lower_leg_joint1: limit lower=0 upper=2.1 effort=300 velocity=0.1 -> lower=0 upper=3.1 effort=300 velocity=0.1; origin xyz=0 0 -0.1 -> xyz=0 0 -0.0623
- joint lower_leg_joint2: limit lower=0 upper=2.1 effort=300 velocity=0.1 -> lower=0 upper=3.1 effort=300 velocity=0.1; origin xyz=0 0 -0.1 -> xyz=0 0 -0.0623
- joint upper_leg_joint00: origin xyz=0 0.07 0 -> xyz=-0.01 0.07 -0.01075
- joint upper_leg_joint01: origin xyz=0 0 0 -> xyz=0 0 -0.004
- joint upper_leg_joint10: origin xyz=0.0606 -0.035 0 -> xyz=0.0656 -0.0263 -0.01075
- joint upper_leg_joint11: origin xyz=0 0 0 -> xyz=0 0 -0.004
- joint upper_leg_joint20: origin xyz=-0.0606 -0.035 0 -> xyz=-0.0556 -0.0437 -0.01075
- joint upper_leg_joint21: origin xyz=0 0 0 -> xyz=0 0 -0.004
